File: ha-usb-switch.kicad_sch (KiCad schematic)
At the start: 9 parts, among them J1 USB4125-GF-A-0190_REVA2, J4 USB1046-XX-XXXX-X-B-X_REVB, Q2 AO3401A, Q3 AO3400A, SW2 SW_SPDT, U1 MOUDLE-SEEEDUINO-XIAO-ESP32C3

Commit message: Add USB C sink pullups
Parts:
- added R4, R5: 56k, Resistor_SMD:R_0603_1608Metric_Pad0.98x0.95mm_HandSolder, symbol Device:R_Small
Connections:
- net +5V: now also R4.2, R5.1
- net at J1.A5 (CC1): now also R4.1
- net at J1.B5 (CC2): now also R5.2
- no-connect marks 15 -> 13
Changed lines of the file:
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@@
+	)
+	(junction
+		(at 101.6 85.09)
+		(diameter 0)
+		(color 0 0 0 0)
+	)
+	(junction
+		(at 93.98 85.09)
+		(diameter 0)
+		(color 0 0 0 0)
 	)
 	(junction
@@
 	)
 	(no_connect
-		(at 107.95 95.25)
-	)
-	(no_connect
-		(at 107.95 92.71)
-	)
-	(no_connect
 		(at 46.99 57.15)
 	)
@@
 	(wire
 		(pts
+			(xy 101.6 85.09) (xy 107.95 85.09)
+		)
+		(stroke
+			(width 0)
+			(type default)
+		)
+	)
+	(wire
+		(pts
 			(xy 96.52 34.29) (xy 102.87 34.29)
 		)
@@
 	(wire
 		(pts
+			(xy 101.6 86.36) (xy 101.6 85.09)
+		)
+		(stroke
+			(width 0)
+			(type default)
+		)
+	)
+	(wire
+		(pts
 			(xy 41.91 87.63) (xy 41.91 90.17)
 		)
@@
 	(wire
 		(pts
+			(xy 101.6 92.71) (xy 101.6 91.44)
+		)
+		(stroke
+			(width 0)
+			(type default)
+		)
+	)
+	(wire
+		(pts
 			(xy 96.52 38.1) (xy 105.41 38.1)
 		)
@@
 	(wire
 		(pts
+			(xy 93.98 91.44) (xy 93.98 95.25)
+		)
+		(stroke
+			(width 0)
+			(type default)
+		)
+	)
+	(wire
+		(pts
 			(xy 45.72 114.3) (xy 50.8 114.3)
 		)
@@
 	(wire
 		(pts
+			(xy 107.95 92.71) (xy 101.6 92.71)
+		)
+		(stroke
+			(width 0)
+			(type default)
+		)
+	)
+	(wire
+		(pts
 			(xy 45.72 106.68) (xy 45.72 114.3)
 		)
@@
 	(wire
 		(pts
+			(xy 93.98 85.09) (xy 93.98 86.36)
+		)
+		(stroke
+			(width 0)
+			(type default)
+		)
+	)
+	(wire
+		(pts
 			(xy 58.42 124.46) (xy 58.42 123.19)
 		)
@@
 	(wire
 		(pts
+			(xy 107.95 85.09) (xy 107.95 87.63)
+		)
+		(stroke
+			(width 0)
+			(type default)
+		)
+	)
+	(wire
+		(pts
 			(xy 72.39 87.63) (xy 72.39 90.17)
 		)
@@
 	(wire
 		(pts
-			(xy 104.14 87.63) (xy 107.95 87.63)
+			(xy 93.98 85.09) (xy 101.6 85.09)
 		)
 		(stroke
@@
 	(wire
 		(pts
+			(xy 93.98 95.25) (xy 107.95 95.25)
+		)
+		(stroke
+			(width 0)
+			(type default)
+		)
+	)
+	(wire
+		(pts
 			(xy 26.67 102.87) (xy 26.67 104.14)
 		)
@@
 	(wire
 		(pts
-			(xy 104.14 86.36) (xy 104.14 87.63)
+			(xy 93.98 82.55) (xy 93.98 85.09)
 		)
 		(stroke
@@
 	)
 	(symbol
+		(lib_id "Device:R_Small")
+		(at 101.6 88.9 180)
+		(unit 1)
+		(exclude_from_sim no)
+		(in_bom yes)
+		(on_board yes)
+		(dnp no)
+		(fields_autoplaced yes)
+		(property "Reference" "R4"
+			(at 103.0986 87.6878 0)
+			(effects
+				(font
+					(size 1.27 1.27)
+				)
+				(justify right)
+			)
+		)
+		(property "Value" "56k"
+			(at 103.0986 90.1121 0)
+			(effects
+				(font
+					(size 1.27 1.27)
+				)
+				(justify right)
+			)
+		)
+		(property "Footprint" "Resistor_SMD:R_0603_1608Metric_Pad0.98x0.95mm_HandSolder"
+			(at 101.6 88.9 0)
+			(effects
+				(font
+					(size 1.27 1.27)
+				)
+				(hide yes)
+			)
+		)
+		(property "Datasheet" "~"
+			(at 101.6 88.9 0)
+			(effects
+				(font
+					(size 1.27 1.27)
+				)
+				(hide yes)
+			)
+		)
+		(property "Description" "Resistor, small symbol"
+			(at 101.6 88.9 0)
+			(effects
+				(font
+					(size 1.27 1.27)
+				)
+				(hide yes)
+			)
+		)
+		(pin "2"
+		)
+		(pin "1"
+		)
+		(instances
+			(project "ha-usb-switch"
+				(path "/20d31bfa-a88e-404e-a379-3f6fa0b30aa5"
+					(reference "R4")
+					(unit 1)
+				)
+			)
+		)
+	)
+	(symbol
 		(lib_name "+5V_1")
 		(lib_id "power:+5V")
@@
 		(lib_name "+5V_1")
 		(lib_id "power:+5V")
-		(at 104.14 86.36 0)
+		(at 93.98 82.55 0)
 		(unit 1)
 		(exclude_from_sim no)
@@
 		(fields_autoplaced yes)
 		(property "Reference" "#PWR03"
-			(at 104.14 90.17 0)
+			(at 93.98 86.36 0)
 			(effects
 				(font
@@
 		)
 		(property "Value" "+5V"
-			(at 104.14 82.2269 0)
+			(at 93.98 78.4169 0)
 			(effects
 				(font
@@
 		)
 		(property "Footprint" ""
-			(at 104.14 86.36 0)
+			(at 93.98 82.55 0)
 			(effects
 				(font
@@
 		)
 		(property "Datasheet" ""
-			(at 104.14 86.36 0)
+			(at 93.98 82.55 0)
 			(effects
 				(font
@@
 		)
 		(property "Description" "Power symbol creates a global label with name \"+5V\""
-			(at 104.14 86.36 0)
+			(at 93.98 82.55 0)
 			(effects
 				(font
@@
 					(unit 1)
 				)
+			)
+		)
+	)
+	(symbol
+		(lib_id "Device:R_Small")
+		(at 93.98 88.9 0)
+		(unit 1)
+		(exclude_from_sim no)
+		(in_bom yes)
+		(on_board yes)
+		(dnp no)
+		(fields_autoplaced yes)
+		(property "Reference" "R5"
+			(at 95.4786 87.6878 0)
+			(effects
+				(font
+					(size 1.27 1.27)
+				)
+				(justify left)
+			)
+		)
+		(property "Value" "56k"
+			(at 95.4786 90.1121 0)
+			(effects
+				(font
+					(size 1.27 1.27)
+				)
+				(justify left)
+			)
+		)
+		(property "Footprint" "Resistor_SMD:R_0603_1608Metric_Pad0.98x0.95mm_HandSolder"
+			(at 93.98 88.9 0)
+			(effects
+				(font
+					(size 1.27 1.27)
+				)
+				(hide yes)
+			)
+		)
+		(property "Datasheet" "~"
+			(at 93.98 88.9 0)
+			(effects
+				(font
+					(size 1.27 1.27)
+				)
+				(hide yes)
+			)
+		)
+		(property "Description" "Resistor, small symbol"
+			(at 93.98 88.9 0)
+			(effects
+				(font
+					(size 1.27 1.27)
+				)
+				(hide yes)
+			)
+		)
+		(pin "2"
+		)
+		(pin "1"
+		)
+		(instances
+			(project "ha-usb-switch"
+				(path "/20d31bfa-a88e-404e-a379-3f6fa0b30aa5"
+					(reference "R5")
+					(unit 1)
+				)
